Commit message: feat: 实现用于四足机器人仿真的 LeapTask 1. 为 12 自由度四足机器人添加了 LeapTask 类，支持特有的奖励函数和腿部功率对称性计算。 2. 创建了 test_leap.py 以验证 LeapTask 的初始化和基本功能。 3. 增强了 helper.py，增加了用于任务配置的命令行参数解析功能。 4. 更新了 Leap.urdf 以对网格文件使用相对路径，从而提高了可移植性。 5. 调整了 hf_util.py 中的日志级别，以提供更好的调试信息。

File: roboverse_data/robots/Leap/urdf/Leap.urdf (robot description, URDF)
Before this commit: robot robot, 18 links, 17 joints
Links:
- link LF_calf: geometry collision mesh filename=../meshes/calf.STL scale=1 1 1; visual mesh filename=../meshes/calf.STL scale=1 1 1
- link LF_hip: geometry collision mesh filename=../meshes/hip.STL scale=1 1 1; visual mesh filename=../meshes/hip.STL scale=1 1 1
- link LF_thigh: geometry collision mesh filename=../meshes/thigh.STL scale=1 1 1; visual mesh filename=../meshes/thigh.STL scale=1 1 1
- link LH_calf: geometry collision mesh filename=../meshes/calf.STL scale=1 1 1; visual mesh filename=../meshes/calf.STL scale=1 1 1
- link LH_hip: geometry collision mesh filename=../meshes/hip.STL scale=1 1 1; visual mesh filename=../meshes/hip.STL scale=1 1 1
- link LH_thigh: geometry collision mesh filename=../meshes/thigh.STL scale=1 1 1; visual mesh filename=../meshes/thigh.STL scale=1 1 1
- link RF_calf: geometry collision mesh filename=../meshes/calf.STL scale=1 1 1; visual mesh filename=../meshes/calf.STL scale=1 1 1
- link RF_hip: geometry collision mesh filename=../meshes/hip.STL scale=1 1 1; visual mesh filename=../meshes/hip.STL scale=1 1 1
- link RF_thigh: geometry collision mesh filename=../meshes/thigh_mirror.STL scale=1 1 1; visual mesh filename=../meshes/thigh_mirror.STL scale=1 1 1
- link RH_calf: geometry collision mesh filename=../meshes/calf.STL scale=1 1 1; visual mesh filename=../meshes/calf.STL scale=1 1 1
- link RH_hip: geometry collision mesh filename=../meshes/hip.STL scale=1 1 1; visual mesh filename=../meshes/hip.STL scale=1 1 1
- link RH_thigh: geometry collision mesh filename=../meshes/thigh_mirror.STL scale=1 1 1; visual mesh filename=../meshes/thigh_mirror.STL scale=1 1 1
- link base: geometry collision mesh filename=../meshes/trunk.STL scale=1 1 1; visual mesh filename=../meshes/trunk.STL scale=1 1 1

Commit message: feat: 更新 Leap 机器人配置并添加 MJCF 与 USD支持 1. 更新了任务配置，以便在 BaseTaskCfg 中初始化 RenderCfg，从而修复了isaacsim仿真报错。 2. 添加了 Leap 机器人的 MJCF 与 USD 模型文件 3. 增强了 LeapCfg，使其包含 Leap 机器人的 MJCF 和 USD 路径。 4. 实现了 URDF 到 USD 的转换脚本，并提供了 Shell 脚本以便于使用。

File: roboverse_data/robots/Leap/urdf/Leap.urdf (robot description, URDF)
Before this commit: robot robot, 18 links, 17 joints
Links:
- link LF_calf: geometry collision mesh filename=/home/ubuntu/RoboVerse/roboverse_data/robots/Leap/meshes/ca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 scale=1 1 1; visual mesh filename=/home/ubuntu/RoboVerse/roboverse_data/robots/Leap/meshes/ca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 scale=1 1 1
- link LF_hip: geometry collision mesh filename=/home/ubuntu/RoboVerse/roboverse_data/robots/Leap/meshes/hi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 scale=1 1 1; visual mesh filename=/home/ubuntu/RoboVerse/roboverse_data/robots/Leap/meshes/hi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 scale=1 1 1
- link LF_thigh: geometry collision mesh filename=/home/ubuntu/RoboVerse/roboverse_data/robots/Leap/meshes/th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 scale=1 1 1; visual mesh filename=/home/ubuntu/RoboVerse/roboverse_data/robots/Leap/meshes/th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 scale=1 1 1
- link LH_calf: geometry collision mesh filename=/home/ubuntu/RoboVerse/roboverse_data/robots/Leap/meshes/ca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 scale=1 1 1; visual mesh filename=/home/ubuntu/RoboVerse/roboverse_data/robots/Leap/meshes/ca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 scale=1 1 1
- link LH_hip: geometry collision mesh filename=/home/ubuntu/RoboVerse/roboverse_data/robots/Leap/meshes/hi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 scale=1 1 1; visual mesh filename=/home/ubuntu/RoboVerse/roboverse_data/robots/Leap/meshes/hi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 scale=1 1 1
- link LH_thigh: geometry collision mesh filename=/home/ubuntu/RoboVerse/roboverse_data/robots/Leap/meshes/th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 scale=1 1 1; visual mesh filename=/home/ubuntu/RoboVerse/roboverse_data/robots/Leap/meshes/th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 scale=1 1 1
- link RF_calf: geometry collision mesh filename=/home/ubuntu/RoboVerse/roboverse_data/robots/Leap/meshes/ca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 scale=1 1 1; visual mesh filename=/home/ubuntu/RoboVerse/roboverse_data/robots/Leap/meshes/ca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 scale=1 1 1
- link RF_hip: geometry collision mesh filename=/home/ubuntu/RoboVerse/roboverse_data/robots/Leap/meshes/hi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 scale=1 1 1; visual mesh filename=/home/ubuntu/RoboVerse/roboverse_data/robots/Leap/meshes/hi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 scale=1 1 1
- link RF_thigh: geometry collision mesh filename=/home/ubuntu/RoboVerse/roboverse_data/robots/Leap/meshes/th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 scale=1 1 1; visual mesh filename=/home/ubuntu/RoboVerse/roboverse_data/robots/Leap/meshes/th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 scale=1 1 1
- link RH_calf: geometry collision mesh filename=/home/ubuntu/RoboVerse/roboverse_data/robots/Leap/meshes/ca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 scale=1 1 1; visual mesh filename=/home/ubuntu/RoboVerse/roboverse_data/robots/Leap/meshes/ca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 scale=1 1 1
- link RH_hip: geometry collision mesh filename=/home/ubuntu/RoboVerse/roboverse_data/robots/Leap/meshes/hi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 scale=1 1 1; visual mesh filename=/home/ubuntu/RoboVerse/roboverse_data/robots/Leap/meshes/hi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 scale=1 1 1
- link RH_thigh: geometry collision mesh filename=/home/ubuntu/RoboVerse/roboverse_data/robots/Leap/meshes/th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 scale=1 1 1; visual mesh filename=/home/ubuntu/RoboVerse/roboverse_data/robots/Leap/meshes/th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 scale=1 1 1
- link base: geometry collision mesh filename=/home/ubuntu/RoboVerse/roboverse_data/robots/Leap/meshes/tr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 scale=1 1 1; visual mesh filename=/home/ubuntu/RoboVerse/roboverse_data/robots/Leap/meshes/tr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 scale=1 1 1
